File: pcb/pcb.kicad_sch (KiCad schematic)
At the start: 11 parts, among them J1 pin_header

Commit message: add pcb
Parts:
- R1, R2, R3, R4, R5, R6, R7, R8: footprint (none) -> Library:100_ohm_resistor
- gave numbers to parts that had none: 1
Changed lines of the file:
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@@
     (pin "3")
   )
-  (symbol (lib_id "components:100_ohm_resistor") (at 119.38 76.2 0) (unit 1)
+  (symbol (lib_name "100_ohm_resistor_2") (lib_id "components:100_ohm_resistor") (at 119.38 76.2 0) (unit 1)
     (in_bom yes) (on_board yes) (fields_autoplaced)
     (property "Reference" "R2" (id 0) (at 119.38 69.85 0))
     (property "Value" "100_ohm_resistor" (id 1) (at 119.38 72.39 0))
-    (property "Footprint" "" (id 2) (at 119.38 76.2 0)
+    (property "Footprint" "Library:100_ohm_resistor" (id 2) (at 119.38 76.2 0)
       (effects (font (size 1.27 1.27)) hide)
     )
@@
     (pin "2")
   )
-  (symbol (lib_id "components:100_ohm_resistor") (at 119.38 87.63 0) (unit 1)
+  (symbol (lib_name "100_ohm_resistor_3") (lib_id "components:100_ohm_resistor") (at 119.38 87.63 0) (unit 1)
     (in_bom yes) (on_board yes)
     (property "Reference" "R3" (id 0) (at 119.38 81.28 0))
     (property "Value" "100_ohm_resistor" (id 1) (at 119.38 83.82 0))
-    (property "Footprint" "" (id 2) (at 119.38 87.63 0)
+    (property "Footprint" "Library:100_ohm_resistor" (id 2) (at 119.38 87.63 0)
       (effects (font (size 1.27 1.27)) hide)
     )
@@
   (symbol (lib_id "components:power_jack_socket") (at 36.83 102.87 0) (unit 1)
     (in_bom yes) (on_board yes) (fields_autoplaced)
-    (property "Reference" "J?" (id 0) (at 36.83 99.06 0)
+    (property "Reference" "J2" (id 0) (at 36.83 99.06 0)
       (effects (font (size 1.27 1.27)) hide)
     )
@@
     (pin "3")
   )
-  (symbol (lib_id "components:100_ohm_resistor") (at 119.38 64.77 0) (unit 1)
+  (symbol (lib_name "100_ohm_resistor_1") (lib_id "components:100_ohm_resistor") (at 119.38 64.77 0) (unit 1)
     (in_bom yes) (on_board yes) (fields_autoplaced)
     (property "Reference" "R1" (id 0) (at 119.38 58.42 0))
     (property "Value" "100_ohm_resistor" (id 1) (at 119.38 60.96 0))
-    (property "Footprint" "" (id 2) (at 119.38 64.77 0)
+    (property "Footprint" "Library:100_ohm_resistor" (id 2) (at 119.38 64.77 0)
       (effects (font (size 1.27 1.27)) hide)
     )
@@
     (pin "2")
   )
-  (symbol (lib_id "components:100_ohm_resistor") (at 119.38 133.35 0) (unit 1)
+  (symbol (lib_name "100_ohm_resistor_7") (lib_id "components:100_ohm_resistor") (at 119.38 133.35 0) (unit 1)
     (in_bom yes) (on_board yes) (fields_autoplaced)
     (property "Reference" "R7" (id 0) (at 119.38 127 0))
     (property "Value" "100_ohm_resistor" (id 1) (at 119.38 129.54 0))
-    (property "Footprint" "" (id 2) (at 119.38 133.35 0)
+    (property "Footprint" "Library:100_ohm_resistor" (id 2) (at 119.38 133.35 0)
       (effects (font (size 1.27 1.27)) hide)
     )
@@
     (pin "2")
   )
-  (symbol (lib_id "components:100_ohm_resistor") (at 119.38 121.92 0) (unit 1)
+  (symbol (lib_name "100_ohm_resistor_6") (lib_id "components:100_ohm_resistor") (at 119.38 121.92 0) (unit 1)
     (in_bom yes) (on_board yes) (fields_autoplaced)
     (property "Reference" "R6" (id 0) (at 119.38 115.57 0))
     (property "Value" "100_ohm_resistor" (id 1) (at 119.38 118.11 0))
-    (property "Footprint" "" (id 2) (at 119.38 121.92 0)
+    (property "Footprint" "Library:100_ohm_resistor" (id 2) (at 119.38 121.92 0)
       (effects (font (size 1.27 1.27)) hide)
     )
@@
     (pin "2")
   )
-  (symbol (lib_id "components:100_ohm_resistor") (at 119.38 110.49 0) (unit 1)
+  (symbol (lib_name "100_ohm_resistor_5") (lib_id "components:100_ohm_resistor") (at 119.38 110.49 0) (unit 1)
     (in_bom yes) (on_board yes) (fields_autoplaced)
     (property "Reference" "R5" (id 0) (at 119.38 104.14 0))
     (property "Value" "100_ohm_resistor" (id 1) (at 119.38 106.68 0))
-    (property "Footprint" "" (id 2) (at 119.38 110.49 0)
+    (property "Footprint" "Library:100_ohm_resistor" (id 2) (at 119.38 110.49 0)
       (effects (font (size 1.27 1.27)) hide)
     )
@@
     (pin "2")
   )
-  (symbol (lib_id "components:100_ohm_resistor") (at 119.38 99.06 0) (unit 1)
+  (symbol (lib_name "100_ohm_resistor_4") (lib_id "components:100_ohm_resistor") (at 119.38 99.06 0) (unit 1)
     (in_bom yes) (on_board yes) (fields_autoplaced)
     (property "Reference" "R4" (id 0) (at 119.38 92.71 0))
     (property "Value" "100_ohm_resistor" (id 1) (at 119.38 95.25 0))
-    (property "Footprint" "" (id 2) (at 119.38 99.06 0)
+    (property "Footprint" "Library:100_ohm_resistor" (id 2) (at 119.38 99.06 0)
       (effects (font (size 1.27 1.27)) hide)
     )
@@
     (property "Reference" "R8" (id 0) (at 119.38 138.43 0))
     (property "Value" "100_ohm_resistor" (id 1) (at 119.38 140.97 0))
-    (property "Footprint" "" (id 2) (at 119.38 144.78 0)
+    (property "Footprint" "Library:100_ohm_resistor" (id 2) (at 119.38 144.78 0)
       (effects (font (size 1.27 1.27)) hide)
     )
@@
     )
     (path "/1e86f799-362b-4148-b112-c90388cb0045"
-      (reference "J?") (unit 1) (value "power_jack_socket") (footprint "Library:power_jack_socket")
+      (reference "J2") (unit 1) (value "power_jack_socket") (footprint "Library:power_jack_socket")
     )
     (path "/2062f576-c723-41ae-b2cb-5cd29c40c3a1"
-      (reference "R1") (unit 1) (value "100_ohm_resistor") (footprint "")
+      (reference "R1") (unit 1) (value "100_ohm_resistor") (footprint "Library:100_ohm_resistor")
     )
     (path "/0a678591-1b8b-4c9a-806c-5fdedd7b2e82"
-      (reference "R2") (unit 1) (value "100_ohm_resistor") (footprint "")
+      (reference "R2") (unit 1) (value "100_ohm_resistor") (footprint "Library:100_ohm_resistor")
     )
     (path "/18850c45-2448-430c-9fe1-508e9ef1d65a"
-      (reference "R3") (unit 1) (value "100_ohm_resistor") (footprint "")
+      (reference "R3") (unit 1) (value "100_ohm_resistor") (footprint "Library:100_ohm_resistor")
     )
     (path "/c6d80819-3e81-4742-b41f-2fa1aec4e839"
-      (reference "R4") (unit 1) (value "100_ohm_resistor") (footprint "")
+      (reference "R4") (unit 1) (value "100_ohm_resistor") (footprint "Library:100_ohm_resistor")
     )
     (path "/9a71deab-c349-4880-9a39-83ceba32d9f6"
-      (reference "R5") (unit 1) (value "100_ohm_resistor") (footprint "")
+      (reference "R5") (unit 1) (value "100_ohm_resistor") (footprint "Library:100_ohm_resistor")
     )
     (path "/8d3aa27e-008c-4b67-bd61-dfdf636263fc"
-      (reference "R6") (unit 1) (value "100_ohm_resistor") (footprint "")
+      (reference "R6") (unit 1) (value "100_ohm_resistor") (footprint "Library:100_ohm_resistor")
     )
     (path "/45d1479d-1e37-40b0-9ab0-dbd809671d8b"
-      (reference "R7") (unit 1) (value "100_ohm_resistor") (footprint "")
+      (reference "R7") (unit 1) (value "100_ohm_resistor") (footprint "Library:100_ohm_resistor")
     )
     (path "/ca4fb951-33c5-41a7-ad60-ef171d3db06f"
-      (reference "R8") (unit 1) (value "100_ohm_resistor") (footprint "")
+      (reference "R8") (unit 1) (value "100_ohm_resistor") (footprint "Library:100_ohm_resistor")
     )
     (path "/05ca308e-df62-4d44-b49f-ec4dc441d2f1"

Commit message: add details to sheets
Other:
- company: (none) -> Francesco Mecatti
- title: (none) -> pcb4fan
Changed lines of the file:
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@@
 (kicad_sch (version 20211123) (generator eeschema)
   (paper "A4")
+  (title_block
+    (title "pcb4fan")
+    (date "2022-01-22")
+    (rev "1.0")
+    (company "Francesco Mecatti")
+  )
   (junction (at 110.49 99.06) (diameter 0) (color 0 0 0 0)
   )
