File: pcb/pcb.kicad_pcb (KiCad board)
At the start: 2 copper layers, 11 parts, among them J1 pin_header, J2 power_jack_socket

Commit message: add 3D model to outfiles
Other:
- board outline added: 56.4 x 49.3 mm
Changed lines of the file:
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@@
       (svguseinch false)
       (svgprecision 6)
-      (excludeedgelayer true)
+      (excludeedgelayer false)
       (plotframeref false)
       (viasonmask false)
@@
       (outputformat 1)
       (mirror false)
-      (drillshape 1)
+      (drillshape 0)
       (scaleselection 1)
       (outputdirectory "")
@@
     )
   )
+  (gr_rect (start 128.99 74.62) (end 185.35 123.92) (layer "Edge.Cuts") (width 0.1) (fill none))
   (gr_rect (start 129.161956 74.793478) (end 185.161956 123.793478) (layer "F.CrtYd") (width 0.05) (fill none))
   (segment (start 146.999456 85.735978) (end 146.999456 77.630978) (width 0.8) (layer "F.Cu") (net 1))
